File: dual-tx-switch/dual-tx-switch.kicad_sch (KiCad schematic)
At the start: 0 parts

Commit message: Crack on with RF detection
Parts:
- added C1: 0.01uF, symbol Device:C_Polarized
- added C2, C5: 0.001uF, symbol Device:C_Polarized
- added C3: 10uF, symbol Device:C_Polarized
- added C4: 1.2pF, symbol Device:C_Polarized
- added D1, D4: CPMD914, symbol Device:D
- added D5, D?: BAS70-04, symbol Device:D
- added J?: XCVR_1, symbol Connector:Conn_Coaxial
- added K?: AZ850-x, Relay_THT:Relay_DPDT_FRT5, symbol Relay:AZ850-x
- added Q1, Q2: 2N7002, Package_TO_SOT_SMD:SOT-23, symbol Transistor_FET:2N7002
- added Q3: MMBT3904, Package_TO_SOT_SMD:SOT-23, symbol Transistor_BJT:MMBT3904
- added R10: 47k, symbol Device:R
- added R7: 1M, symbol Device:R_Potentiometer
- added R8: 2.2k, symbol Device:R
- added R9: 10k, symbol Device:R
Connections:
- new net: D1.2 (A), K?.10, Q1.3 (D), Q2.3 (D)
- new net: C5.1, D?.1 (K), Q3.1 (B), R10.1
- new net: J?.1 (In), K?.3
- new net: R7.1, R9.1
- new net: C3.1, D4.2 (A), Q1.1 (G), Q2.1 (G), Q3.3 (C), R9.2
- new net: C4.1, D5.1 (K), D?.2 (A)
- new net: C4.2, K?.8
- new net: C2.1, D4.1 (K), R8.2
- new net: K?.2, K?.9
- new net +12V: C1.1, D1.1 (K), K?.1, R7.2, R7.3, R8.1
- new net GND: C1.2, C2.2, C3.2, C5.2, D5.2 (A), Q1.2 (S), Q2.2 (S), Q3.2 (E), R10.2
